File: Stage flood sensor/Stage flood sensor.kicad_pcb (KiCad board)
At the start: 4 copper layers, 100 x 100 mm, 2 parts, among them J1 Conn_01x01_Female, J2 Conn_01x01_Female

Commit message: Ordered
Parts:
- added C1: 10 µF, Custom footprints:0603 Passthrough capacitor, B.Cu at (100.5, 137.2)
- added JP1: Jumper_3_Open, Jumper:SolderJumper-3_P2.0mm_Open_TrianglePad1.0x1.5mm_NumberLabels, B.Cu at (103.0, 135.8)
- added R2: 1k, Resistor_SMD:R_0603_1608Metric, B.Cu at (100.5, 134.3)
- added REF**: OSHW-Logo_11.4x12mm_SilkScreen, Symbol:OSHW-Logo_11.4x12mm_SilkScreen, B.Cu at (63.1, 58.1)
Connections:
- J1 pad 1: /Sense -> Net-(J1-Pin_1)
Routing:
- net Net-(J1-Pin_1): track 0.00 -> 12.8 mm
- net Net-(JP1-C): track 0.00 -> 3.83 mm
- net GND: track 6527.9 -> 6529.9 mm, vias 651 -> 648
Other:
- board text added: "+"
- board text added: "-"
- board text added: "RC Filter"
- board text added: "Stage Flood Sensor Designed by: Benjamin E. Smith Funded by: NIH P30EY003176 https://github.com/Llamero/Stage_flood_sensor"
