File: Stage flood sensor/Stage flood sensor.kicad_sch (KiCad schematic)
At the start: 5 parts, among them J1 Conn_01x01_Female, J2 Conn_01x01_Female

Commit message: Ordered
Parts:
- C1: value Filter_EMI_C -> 10 µF; footprint (none) -> Custom footprints:0603 Passthrough capacitor; Part # (none) -> YFF18PH0J106MT00HE
- R2: value R -> 1k; footprint (none) -> Resistor_SMD:R_0603_1608Metric; Part # (none) -> RNCP0603FTD1K00
Changed lines of the file:
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@@
   (symbol (lib_id "Device:Filter_EMI_C") (at 97.79 60.96 0) (mirror y) (unit 1)
     (in_bom yes) (on_board yes) (dnp no)
-    (property "Reference" "C1" (at 96.52 53.34 0)
+    (property "Reference" "C1" (at 97.79 53.34 0)
       (effects (font (size 1.27 1.27)))
     )
-    (property "Value" "Filter_EMI_C" (at 96.52 55.88 0)
+    (property "Value" "10 µF" (at 97.79 55.88 0)
       (effects (font (size 1.27 1.27)))
     )
-    (property "Footprint" "" (at 97.79 60.96 90)
+    (property "Footprint" "Custom footprints:0603 Passthrough capacitor" (at 97.79 60.96 90)
       (effects (font (size 1.27 1.27)) hide)
     )
     (property "Datasheet" "http://www.murata.com/~/media/webrenewal/support/library/catalog/products/emc/emifil/c31e.ashx?la=en-gb" (at 97.79 60.96 90)
+      (effects (font (size 1.27 1.27)) hide)
+    )
+    (property "Part #" "YFF18PH0J106MT00HE" (at 97.79 60.96 0)
       (effects (font (size 1.27 1.27)) hide)
     )
@@
   )
   (symbol (lib_id "Device:R") (at 106.68 58.42 270) (mirror x) (unit 1)
-    (in_bom yes) (on_board yes) (dnp no) (fields_autoplaced)
-    (property "Reference" "R2" (at 106.68 54.3941 90)
+    (in_bom yes) (on_board yes) (dnp no)
+    (property "Reference" "R2" (at 106.68 55.88 90)
       (effects (font (size 1.27 1.27)))
     )
-    (property "Value" "R" (at 106.68 56.3151 90)
+    (property "Value" "1k" (at 106.68 58.42 90)
       (effects (font (size 1.27 1.27)))
     )
-    (property "Footprint" "" (at 106.68 60.198 90)
+    (property "Footprint" "Resistor_SMD:R_0603_1608Metric" (at 106.68 60.198 90)
       (effects (font (size 1.27 1.27)) hide)
     )
@@
       (effects (font (size 1.27 1.27)) hide)
     )
+    (property "Part #" "RNCP0603FTD1K00" (at 106.68 58.42 90)
+      (effects (font (size 1.27 1.27)) hide)
+    )
